Commit message: Expand README with gallery, architecture diagrams and procedures
- Gallery: robot close-up and Nav2 navigation view rendered from the
  simulation, plus world, corridor and SLAM map images
- Mermaid diagrams of the ROS node graph and TF tree
- Step-by-step installation, mapping, navigation and headless usage
- Customising, verification commands, troubleshooting table,
  measured performance and engineering notes
- Gazebo materials for wheels, LiDAR and camera (Gazebo ignores URDF
  colours); visual only

File: src/skid_steer_amr/urdf/camera.xacro (robot description, xacro)
@@ -32,4 +32,7 @@
     </inertial>
   </link>
+  <gazebo reference="camera_link">
+    <material>Gazebo/FlatBlack</material>   <!-- Gazebo ignores URDF colours -->
+  </gazebo>
   <joint name="camera_joint" type="fixed">
     <parent link="base_link"/>

File: src/skid_steer_amr/urdf/lidar.xacro (robot description, xacro)
@@ -23,4 +23,5 @@
   </joint>
   <gazebo reference="lidar_link">
+    <material>Gazebo/DarkGrey</material>
     <sensor name="lidar" type="ray">
       <always_on>true</always_on>

File: src/skid_steer_amr/urdf/robot_core.xacro (robot description, xacro)
@@ -75,4 +75,5 @@
          direction. Low sideways friction lets the robot skid when turning. -->
     <gazebo reference="${name}_link">
+      <material>Gazebo/FlatBlack</material>   <!-- Gazebo ignores URDF colours -->
       <mu1>0.3</mu1>
       <mu2>1.0</mu2>
