Commit message: Add base_footprint frame, fix RViz robot model and views

File: src/skid_steer_amr/urdf/gazebo_control.xacro (robot description, xacro)
@@ -7,5 +7,5 @@
       subscribes: /cmd_vel (geometry_msgs/Twist)
       publishes:  /odom    (nav_msgs/Odometry), wheel TFs
-    odom -> base_link TF is published by the EKF, not by this plugin.
+    odom -> base_footprint TF is published by the EKF, not by this plugin.
   -->
   <gazebo>
@@ -34,5 +34,5 @@
       <odometry_topic>odom</odometry_topic>
       <odometry_frame>odom</odometry_frame>
-      <robot_base_frame>base_link</robot_base_frame>
+      <robot_base_frame>base_footprint</robot_base_frame>
     </plugin>
   </gazebo>

File: src/skid_steer_amr/urdf/lidar.xacro (robot description, xacro)
@@ -26,5 +26,5 @@
     <sensor name="lidar" type="ray">
       <always_on>true</always_on>
-      <visualize>true</visualize>
+      <visualize>false</visualize>  <!-- true draws the rays in Gazebo -->
       <update_rate>10</update_rate>
       <ray>

File: src/skid_steer_amr/urdf/robot_core.xacro (robot description, xacro)
@@ -9,4 +9,15 @@
   <xacro:property name="wheel_y"      value="0.16"/>  <!-- joint position, left (+) / right (-) -->
   <xacro:property name="wheel_offset" value="0.02"/>  <!-- wheel centre sits this far outboard of its joint -->
+  <!-- ======================================================= -->
+  <!--  base_footprint: robot frame on the floor, directly below -->
+  <!--  the chassis (REP-105). EKF, AMCL, SLAM and Nav2 track    -->
+  <!--  this frame; base_link sits at wheel-axle height above it -->
+  <!-- ======================================================= -->
+  <link name="base_footprint"/>
+  <joint name="base_footprint_joint" type="fixed">
+    <parent link="base_footprint"/>
+    <child link="base_link"/>
+    <origin xyz="0 0 ${wheel_radius}" rpy="0 0 0"/>
+  </joint>
   <!-- ======================================================= -->
   <!--  Chassis                                                 -->
